File: KAKATA_MOD_FUNCIONES/KAKATA_MOD_FUNCIONES.kicad_pcb (KiCad board)
At the start: 4 copper layers, 55.7 x 46.6 mm, 29 parts, among them U1 ESP32-S3-WROOM-1(N16R8), U10 DB125-2.54-4P-GN, U11 DB125-2.54-4P-GN, U12 DB125-2.54-4P-GN, U13 DB125-2.54-4P-GN, U14 DB125-2.54-4P-GN, U2 PSC-1608U52GC-G4, U3 PSC-1608U52GC-G4, U4 PSC-1608U52GC-G4, U5 PSC-1608U52GC-G4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

Commit message: Base hecha
Parts:
- removed U9: DB125-3.5-2P-GN-S, EasyEDA:CONN-TH_2P-P3.50_L7.4-W7.0
- added CN1: HX JN1.27-2X3 TP H4.9, EasyEDA:CONN-SMD_6P-P1.27-LS5.8, F.Cu at (88.8, 37.0)
- added R12: 10K, PCM_Resistor_SMD_AKL:R_0603_1608Metric, F.Cu at (119.8, 59.0)
- R1: value R_0603 -> 10K
- moved R4 27.8 mm to (119.9, 57.0)
- moved U7 26.2 mm to (86.3, 64.8)
- moved U12 18.8 mm to (96.5, 68.0)
- moved U2 18.6 mm to (126.4, 55.8), turned to 180 degrees
- moved U10 18.6 mm to (108.0, 68.0), turned to 180 degrees
- moved U14 18.2 mm to (119.5, 68.0), turned to 180 degrees
- moved U3 17.6 mm to (126.3, 53.8), turned to 180 degrees
- moved U4 17.0 mm to (126.4, 51.8), turned to 180 degrees
- moved U5 16.8 mm to (126.3, 49.8), turned to 180 degrees
- moved R5 10.9 mm to (101.3, 61.3), turned to 90 degrees
- moved U11 10.1 mm to (87.3, 54.8), turned to 90 degrees
- moved H5 9.78 mm to (135.3, 48.0)
- moved H7 4.67 mm to (135.3, 74.0)
- moved H8 4.00 mm to (81.3, 74.0)
- moved U8 2.05 mm to (86.8, 44.8), turned to 90 degrees
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Connections:
- net Net-(U1-EN) renamed /EN
- U1 pad 27: unconnected-(U1-IO0-Pad27) -> /BOOT
- U1 pad 28: /I2C_SCL1 -> /I2C_SCL_1
- U1 pad 36: unconnected-(U1-RXD0-Pad36) -> /ESP_RXD
- U1 pad 37: unconnected-(U1-TXD0-Pad37) -> /ESP_TXD
- U11 pad 1: /I2C_SDA_1 -> +3.3V
- U11 pad 2: /I2C_SCL1 -> /I2C_SDA_1
- U11 pad 3: unconnected-(U11-Pad3) -> /I2C_SCL_1
Routing:
- net /I2C1_D0: track 34.2 -> 0.00 mm, vias 1 -> 0
- net /I2C1_D1: track 34.0 -> 0.00 mm, vias 1 -> 0
- net Net-(U5-A): track 18.2 -> 0.00 mm
- net Net-(U4-A): track 17.8 -> 0.00 mm
- net Net-(U3-A): track 17.6 -> 0.00 mm
- net Net-(U2-A): track 16.3 -> 0.00 mm
- net /OD: track 4.42 -> 0.00 mm, vias 1 -> 0
- net /OC: track 4.36 -> 0.00 mm, vias 1 -> 0
- net +3.3V: track 3.90 -> 0.00 mm, vias 8 -> 0
- net /EN: track 3.32 -> 0.00 mm
- net GND: track 3.04 -> 0.00 mm, vias 34 -> 0
- net /PWM1: track 2.96 -> 0.00 mm, vias 1 -> 0
- net /PH_LED: track 2.63 -> 0.00 mm
- net /CO^{2}_LED: track 2.41 -> 0.00 mm
- net /PWM0: track 2.31 -> 0.00 mm, vias 1 -> 0
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- removed copper zone on F.Cu, net +3.3V
Other:
- board size 55.7 x 46.6 mm -> 57.7 x 42.6 mm
- board text added: "3.3V"
- board text added: "EN TX RX"
- board text added: "ENA"
- board text added: "ENB"
- board text added: "PWM1"
- board text added: "VDD GND BOOT"
- board text removed: "+3.3V"

Commit message: hot_fix_Done
Parts:
- moved R10 3.48 mm to (96.6, 45.0)
- moved R1 1.88 mm to (96.6, 43.0)
- moved R3 1.43 mm to (96.6, 49.0)
- moved R2 1.23 mm to (96.6, 51.0)
- moved C1 0.75 mm to (96.6, 40.8), turned to 0 degrees
- moved R11 0.34 mm to (96.6, 47.0)
Changed lines of the file:
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@@
 	(footprint "PCM_Resistor_SMD_AKL:R_0603_1608Metric"
 		(layer "F.Cu")
-		(at 96.5 46.7 180)
+		(at 96.6 47.025 180)
 		(descr "Resistor SMD 0603 (1608 Metric), square (rectangular) end terminal, IPC_7351 nominal, (Body size source: IPC-SM-782 page 72, https://www.pcb-3d.com/wordpress/wp-content/uploads/ipc-sm-782a_amendment_1_and_2.pdf), Alternate KiCad Library")
 		(tags "resistor")
@@
 	(footprint "PCM_Resistor_SMD_AKL:R_0603_1608Metric"
 		(layer "F.Cu")
-		(at 96.5 48.5 180)
+		(at 96.6 45.025 180)
 		(descr "Resistor SMD 0603 (1608 Metric), square (rectangular) end terminal, IPC_7351 nominal, (Body size source: IPC-SM-782 page 72, https://www.pcb-3d.com/wordpress/wp-content/uploads/ipc-sm-782a_amendment_1_and_2.pdf), Alternate KiCad Library")
 		(tags "resistor")
@@
 	(footprint "PCM_Resistor_SMD_AKL:R_0603_1608Metric"
 		(layer "F.Cu")
-		(at 96.5 52.25)
+		(at 96.6 51.025)
 		(descr "Resistor SMD 0603 (1608 Metric), square (rectangular) end terminal, IPC_7351 nominal, (Body size source: IPC-SM-782 page 72, https://www.pcb-3d.com/wordpress/wp-content/uploads/ipc-sm-782a_amendment_1_and_2.pdf), Alternate KiCad Library")
 		(tags "resistor")
@@
 	(footprint "PCM_Resistor_SMD_AKL:R_0603_1608Metric"
 		(layer "F.Cu")
-		(at 96.5 50.45)
+		(at 96.6 49.025)
 		(descr "Resistor SMD 0603 (1608 Metric), square (rectangular) end terminal, IPC_7351 nominal, (Body size source: IPC-SM-782 page 72, https://www.pcb-3d.com/wordpress/wp-content/uploads/ipc-sm-782a_amendment_1_and_2.pdf), Alternate KiCad Library")
 		(tags "resistor")
@@
 	(footprint "PCM_Resistor_SMD_AKL:R_0603_1608Metric"
 		(layer "F.Cu")
-		(at 96.5 44.9)
+		(at 96.6 43.025)
 		(descr "Resistor SMD 0603 (1608 Metric), square (rectangular) end terminal, IPC_7351 nominal, (Body size source: IPC-SM-782 page 72, https://www.pcb-3d.com/wordpress/wp-content/uploads/ipc-sm-782a_amendment_1_and_2.pdf), Alternate KiCad Library")
 		(tags "resistor")
@@
 	(footprint "PCM_Capacitor_SMD_AKL:C_0603_1608Metric"
 		(layer "F.Cu")
-		(at 97.25 41.15 -90)
+		(at 96.6 40.775)
 		(descr "Capacitor SMD 0603 (1608 Metric), square (rectangular) end terminal, IPC_7351 nominal, (Body size source: IPC-SM-782 page 76, https://www.pcb-3d.com/wordpress/wp-content/uploads/ipc-sm-782a_amendment_1_and_2.pdf), Alternate KiCad Library")
 		(tags "capacitor")
 		(property "Reference" "C1"
-			(at 1.25 1.75 0)
+			(at -2.75 0.25 180)
 			(layer "F.SilkS")
 			(effects
@@
 		)
 		(property "Value" "C_0603"
-			(at 0 1.43 90)
+			(at 0 1.43 0)
 			(layer "F.Fab")
 			(hide yes)
@@
 		)
 		(property "Datasheet" "~"
-			(at 0 0 90)
+			(at 0 0 0)
 			(layer "F.Fab")
 			(hide yes)
@@
 		)
 		(property "Description" "SMD 0603 MLCC capacitor, Alternate KiCad Library"
-			(at 0 0 90)
+			(at 0 0 0)
 			(layer "F.Fab")
 			(hide yes)
@@
 		)
 		(fp_line
-			(start -1.48 0.73)
-			(end -1.48 -0.73)
+			(start -1.48 -0.73)
+			(end 1.48 -0.73)
 			(stroke
 				(width 0.05)
@@
 		)
 		(fp_line
-			(start 1.48 0.73)
-			(end -1.48 0.73)
+			(start -1.48 0.73)
+			(end -1.48 -0.73)
 			(stroke
 				(width 0.05)
@@
 		)
 		(fp_line
-			(start -1.48 -0.73)
-			(end 1.48 -0.73)
+			(start 1.48 -0.73)
+			(end 1.48 0.73)
 			(stroke
 				(width 0.05)
@@
 		)
 		(fp_line
-			(start 1.48 -0.73)
-			(end 1.48 0.73)
+			(start 1.48 0.73)
+			(end -1.48 0.73)
 			(stroke
 				(width 0.05)
@@
 		)
 		(fp_line
-			(start -0.8 0.4)
-			(end -0.8 -0.4)
+			(start -0.8 -0.4)
+			(end 0.8 -0.4)
 			(stroke
 				(width 0.1)
@@
 		)
 		(fp_line
-			(start 0.8 0.4)
-			(end -0.8 0.4)
+			(start -0.8 0.4)
+			(end -0.8 -0.4)
 			(stroke
 				(width 0.1)
@@
 		)
 		(fp_line
-			(start -0.8 -0.4)
-			(end 0.8 -0.4)
+			(start 0.8 -0.4)
+			(end 0.8 0.4)
 			(stroke
 				(width 0.1)
@@
 		)
 		(fp_line
-			(start 0.8 -0.4)
-			(end 0.8 0.4)
+			(start 0.8 0.4)
+			(end -0.8 0.4)
 			(stroke
 				(width 0.1)
@@
 		)
 		(fp_text user "${REFERENCE}"
-			(at 0.8 0 90)
+			(at 0.8 0 0)
 			(layer "F.Fab")
 			(effects
@@
 		)
 		(pad "1" smd roundrect
-			(at -0.775 0 270)
+			(at -0.775 0)
 			(size 0.9 0.95)
 			(layers "F.Cu" "F.Mask" "F.Paste")
@@
 		)
 		(pad "2" smd roundrect
-			(at 0.775 0 270)
+			(at 0.775 0)
 			(size 0.9 0.95)
 			(layers "F.Cu" "F.Mask" "F.Paste")
